File: logging.kicad_sch (KiCad schematic)
At the start: 2 parts, among them J2 Micro_SD_Card, U2 RFM69HW

Commit message: Update references and switch to higher power MOSFETS
Parts:
- renumbered U2 to U1
Changed lines of the file:
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@@
 		(dnp no)
 		(fields_autoplaced yes)
-		(property "Reference" "U2"
+		(property "Reference" "U1"
 			(at 107.5533 93.98 0)
 			(effects
@@
 			(project "rocket"
 				(path "/d94d1fd0-ec09-478b-a1a4-3306111fc872/8ffc271b-b77c-4862-a5e5-6c3b3e515885"
-					(reference "U2")
+					(reference "U1")
 					(unit 1)
 				)

Commit message: External antenna
Parts:
- added J1: Conn_Coaxial, Connector_Coaxial:BNC_Amphenol_031-5539_Vertical, symbol Connector:Conn_Coaxial
Connections:
- net VSS: now also J1.2 (Ext)
- net at U1.10 (ANA): now also J1.1 (In)
- no-connect marks 10 -> 9
Changed lines of the file:
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@@
+	)
+	(junction
+		(at 129.54 106.68)
+		(diameter 0)
+		(color 0 0 0 1)
 	)
 	(junction
@@
 	)
 	(no_connect
-		(at 143.51 101.6)
-	)
-	(no_connect
 		(at 92.71 114.3)
 	)
@@
 	(wire
 		(pts
+			(xy 129.54 106.68) (xy 129.54 121.92)
+		)
+		(stroke
+			(width 0)
+			(type default)
+			(color 0 0 0 1)
+		)
+	)
+	(wire
+		(pts
 			(xy 73.66 60.96) (xy 73.66 90.17)
 		)
@@
 	(wire
 		(pts
+			(xy 123.19 106.68) (xy 129.54 106.68)
+		)
+		(stroke
+			(width 0)
+			(type default)
+			(color 0 0 0 1)
+		)
+	)
+	(wire
+		(pts
 			(xy 86.36 71.12) (xy 83.82 71.12)
 		)
@@
 	(wire
 		(pts
-			(xy 129.54 82.55) (xy 129.54 121.92)
-		)
-		(stroke
-			(width 0)
-			(type default)
-			(color 0 0 0 1)
-		)
-	)
-	(wire
-		(pts
-			(xy 118.11 101.6) (xy 143.51 101.6)
-		)
-		(stroke
-			(width 0)
-			(type default)
+			(xy 129.54 82.55) (xy 129.54 106.68)
+		)
+		(stroke
+			(width 0)
+			(type default)
+			(color 0 0 0 1)
 		)
 	)
@@
 					(unit 1)
 				)
+			)
+		)
+	)
+	(symbol
+		(lib_id "Connector:Conn_Coaxial")
+		(at 123.19 101.6 0)
+		(unit 1)
+		(exclude_from_sim no)
+		(in_bom yes)
+		(on_board yes)
+		(dnp no)
+		(fields_autoplaced yes)
+		(property "Reference" "J1"
+			(at 127 100.6231 0)
+			(effects
+				(font
+					(size 1.27 1.27)
+				)
+				(justify left)
+			)
+		)
+		(property "Value" "Conn_Coaxial"
+			(at 127 103.1631 0)
+			(effects
+				(font
+					(size 1.27 1.27)
+				)
+				(justify left)
+			)
+		)
+		(property "Footprint" "Connector_Coaxial:BNC_Amphenol_031-5539_Vertical"
+			(at 123.19 101.6 0)
+			(effects
+				(font
+					(size 1.27 1.27)
+				)
+				(hide yes)
+			)
+		)
+		(property "Datasheet" "~"
+			(at 123.19 101.6 0)
+			(effects
+				(font
+					(size 1.27 1.27)
+				)
+				(hide yes)
+			)
+		)
+		(property "Description" "coaxial connector (BNC, SMA, SMB, SMC, Cinch/RCA, LEMO, ...)"
+			(at 123.19 101.6 0)
+			(effects
+				(font
+					(size 1.27 1.27)
+				)
+				(hide yes)
+			)
+		)
+		(pin "1"
+		)
+		(pin "2"
+		)
+		(instances
+			(project ""
+				(path "/d94d1fd0-ec09-478b-a1a4-3306111fc872/8ffc271b-b77c-4862-a5e5-6c3b3e515885"
+					(reference "J1")
+					(unit 1)
+				)
