File: rocket.kicad_pcb (KiCad board)
At the start: 2 copper layers, 19 parts, among them J2 Micro_SD_Card, U1 RFM69HW, U2 BMP390, U3 ICM-42670-P, U4 TPS62056DGS, U5 TLP3544, U6 TLP3544

Commit message: PCB improvement
Parts:
- moved U6 53.7 mm to (125.2, 104.5)
- moved U2 48.2 mm to (59.6, 120.8)
- moved U3 45.1 mm to (60.1, 116.7)
- moved U5 44.0 mm to (125.2, 114.0)
- moved H6 42.7 mm to (138.5, 103.0)
- moved J2 39.7 mm to (73.5, 102.1)
- moved L1 39.0 mm to (127.1, 95.1), turned to 0 degrees
- moved C2 37.9 mm to (132.0, 84.5), turned to 90 degrees
- moved U4 37.4 mm to (127.1, 84.6), turned to 90 degrees
- moved H3 31.5 mm to (138.5, 95.5)
- moved C1 31.3 mm to (127.1, 72.6), turned to 0 degrees
- moved R1 30.5 mm to (118.5, 120.0)
- moved H5 29.8 mm to (138.5, 110.5)
- moved R2 28.0 mm to (118.5, 117.5)
- moved H1 25.5 mm to (123.6, 78.1), turned to 90 degrees
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Routing:
- net /Power circuitry/7.4V: track 19.1 -> 80.9 mm
- net /Power circuitry/BGND: track 20.6 -> 62.5 mm
- net Net-(R2-Pad2): track 0.00 -> 16.7 mm
- net Net-(R1-Pad2): track 0.00 -> 8.88 mm
- net Net-(H4-Pad1): track 0.00 -> 7.36 mm
- net Net-(H6-Pad1): track 0.00 -> 6.29 mm
- net Net-(U4-SW): track 11.2 -> 14.5 mm
- net Net-(A1-GPIO17): track 0.00 -> 2.75 mm
- net Net-(A1-GPIO16): track 0.00 -> 2.73 mm
- net /Power circuitry/PGND: track 56.6 -> 58.6 mm, vias 0 -> 2
- net /Data Logging/VDD: track 43.0 -> 44.6 mm
- added copper zone on F.Cu, net /Power circuitry/BGND

Commit message: External antenna
Parts:
- added J1: Conn_Coaxial, Connector_Coaxial:BNC_Amphenol_031-5539_Vertical, F.Cu at (83.5, 95.0)
- moved J2 17.3 mm to (85.0, 115.0), turned to 180 degrees
- moved U1 7.62 mm to (79.0, 78.5)
Connections:
- U1 pad 10: unconnected-(U1-ANA-Pad10) -> Net-(J1-In)
Routing:
- net /Data Logging/SCLK: track 0.00 -> 60.6 mm, vias 0 -> 1
- net /Data Logging/VDD: track 44.6 -> 98.7 mm
- net /Data Logging/MOSI: track 0.00 -> 51.7 mm, vias 0 -> 1
- net /Data Logging/MISO: track 0.00 -> 47.6 mm, vias 0 -> 1
- net /Data Logging/CS1: track 0.00 -> 46.4 mm, vias 0 -> 1
- net /Data Logging/VSS: track 0.00 -> 36.9 mm
- net /Data Logging/CS2: track 0.00 -> 21.2 mm
- net Net-(J1-In): track 0.00 -> 13.9 mm
