File: rocket.kicad_sch (KiCad schematic)
At the start: 9 parts, among them U5 TLP3544, U6 TLP3544

Commit message: Add additional features
Parts:
- added BT1: Battery_Cell, Battery:BatteryClip_Keystone_54_D16-19mm, symbol Device:Battery_Cell
- added BZ1: Buzzer, Buzzer_Beeper:Buzzer_15x7.5RM7.6, symbol Device:Buzzer
- added D1: PWR, LED_SMD:LED_0201_0603Metric, symbol Device:LED
- added D2: RDY, LED_SMD:LED_0201_0603Metric, symbol Device:LED
- added D3: LND, LED_SMD:LED_0201_0603Metric, symbol Device:LED
- added D4: 1N4148WT, Diode_SMD:D_SOD-523, symbol Diode:1N4148WT
- added J3: Conn_Coaxial, Connector_Coaxial:BNC_Amphenol_031-5539_Vertical, symbol Connector:Conn_Coaxial
- added R3, R4, R5: 43Ω, Resistor_SMD:R_0201_0603Metric, symbol Device:R
- added U7: RXM-GPS-RM, RF_GPS:Linx_RXM-GPS, symbol RF_GPS:RXM-GPS-RM
Connections:
- net Data Logging/VDD: now also D1.2 (A)
- net Data Logging/VSS: now also BT1.2 (-), BZ1.2 (-), J3.2 (Ext), R3.2, U7.18 (GND), U7.20 (GND), U7.21 (GND), U7.22 (GND)
- net Power circuitry/PGND: now also R4.2, R5.2, U7.12 (VCC), U7.8 (~{RESET})
- net at A1.19 (GPIO14): now also U7.3 (1PPS)
- net at A1.20 (GPIO15): now also BZ1.1 (+)
- net at A1.25 (GPIO19): now also D2.2 (A)
- net at A1.26 (GPIO20): now also D3.2 (A)
- net at A1.27 (GPIO21): now also U7.5 (RX)
- net at A1.29 (GPIO22): now also U7.4 (TX)
- new net: J3.1 (In), U7.19 (RFIN)
- new net: D2.1 (K), R4.1
- new net: D4.1 (K), U7.11 (VBCKUP)
- new net: BT1.1 (+), D4.2 (A)
- new net: D3.1 (K), R5.1
- new net: D1.1 (K), R3.1
